Commit message: updated controller

File: arduinobot_description/urdf/arduinobot.urdf.xacro (robot description, xacro)
@@ -1,4 +1,5 @@
 <?xml version="1.0"?>
 <robot xmlns:xacro="http://www.ros.org/wiki/xacro" name="arduinobot">
+    <xacro:arg name="is_sim" default="true"/>
     <xacro:include filename="$(find arduinobot_description)/urdf/arduinobot_gazebo.xacro"/>
     <xacro:include filename="$(find arduinobot_description)/urdf/arduinobot_ros2_control.xacro"/>
@@ -37,5 +38,5 @@
         </collision>
     </link>
-    <joint name="virtual_link" type="fixed">
+    <joint name="virtual_joint" type="fixed">
         <parent link="world"/>
         <child link="base_link"/>

File: arduinobot_description/urdf/arduinobot_ros2_control.xacro (robot description, xacro)
@@ -3,7 +3,23 @@
     <xacro:property name="PI" value="3.14159"/>
     <ros2_control name ="RobotSystem" type ="system">
-        <hardware>
-            <plugin>gazebo_ros2_control/GazeboSystem</plugin>
-        </hardware>
+        <xacro:if value="$(arg is_sim)">
+            <hardware>
+                <plugin>gazebo_ros2_control/GazeboSystem</plugin>
+            </hardware>
+            <joint name="joint_5">
+                <param name="mimic">joint_4</param>
+                <param name="multiplier">-1</param>
+                <command_interface name="position">
+                    <param name="min">0.0</param>
+                    <param name="max">${PI/2}</param>
+                </command_interface>
+            </joint>
+        </xacro:if>
+        <xacro:unless value="$(arg is_sim)">
+            <hardware>
+                <plugin>arduinobot_controller/ArduinobotInterface</plugin>
+                <param name="port">/dev/ttyACM0</param>
+            </hardware>
+        </xacro:unless>
         <joint name="joint_1">
             <command_interface name="position">
@@ -34,13 +50,4 @@
             <state_interface name="position"/>
         </joint>
-        <joint name="joint_5">
-            <param name="mimic">joint_4</param>
-            <param name="multiplier">-1</param>
-            <command_interface name="position">
-                <param name="min">0.0</param>
-                <param name="max">${PI/2}</param>
-            </command_interface>
-            <state_interface name="position"/>
-        </joint>
     </ros2_control>
 </robot>
